File: EDA/DB19_IDC20/DB19_IDC20.kicad_pcb (KiCad board)
At the start: 2 copper layers, 40 x 20 mm, 2 parts, among them J1 Conn_02x10_Odd_Even, J2 DB19_Female

Commit message: renamed adapter
Other:
- board text added: "TASHTWENTY TINY ADAPTER"
- board text removed: "TASHTWENTY MINI ADAPTER"
