File: EDA/DB19_IDC20/DB19_IDC20.kicad_pcb (KiCad board)
At the start: 2 copper layers, 40 x 20 mm, 2 parts, among them J1 Conn_02x10_Odd_Even, J2 DB19_Female

Commit message: minor fixes for production
Other:
- board text added: "JLCJLCJLCJLC"
Changed lines of the file:
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@@
-(kicad_pcb (version 20171130) (host pcbnew "(5.1.9-0-10_14)")
+(kicad_pcb (version 20171130) (host pcbnew "(5.1.12-1-10_14)")
   (general
     (thickness 1.6)
-    (drawings 14)
+    (drawings 15)
     (tracks 44)
     (zones 0)
@@
     (visible_elements FFFFFF7F)
     (pcbplotparams
-      (layerselection 0x010fc_ffffffff)
+      (layerselection 0x010f0_ffffffff)
       (usegerberextensions false)
       (usegerberattributes true)
@@
       (outputformat 1)
       (mirror false)
-      (drillshape 1)
+      (drillshape 0)
       (scaleselection 1)
       (outputdirectory ""))
@@
     (pad 3 thru_hole circle (at 0 2.54 90) (size 1.7 1.7) (drill 1) (layers *.Cu *.Mask)
       (net 2 GND))
-    (pad 1 thru_hole roundrect (at 0 0 90) (size 1.7 1.7) (drill 1) (layers *.Cu *.Mask) (roundrect_rratio 0.147059)
+    (pad 1 thru_hole roundrect (at 0 0 90) (size 1.7 1.7) (drill 1) (layers *.Cu *.Mask) (roundrect_rratio 0.1470588235294118)
       (net 2 GND))
     (model ${KISYS3DMOD}/Connector_IDC.3dshapes/IDC-Header_2x10_P2.54mm_Vertical.wrl
@@
     )
   )
+  (gr_text JLCJLCJLCJLC (at 120 110) (layer B.SilkS)
+    (effects (font (size 1 1) (thickness 0.15)) (justify mirror))
+  )
   (gr_text 10 (at 136 118) (layer F.SilkS)
     (effects (font (size 1.5 1.5) (thickness 0.3)))
@@
     (effects (font (size 1.5 1.5) (thickness 0.3)) (justify mirror))
   )
-  (gr_text 68kmla.org (at 120 112) (layer B.SilkS)
+  (gr_text 68kmla.org (at 120 113) (layer B.SilkS)
     (effects (font (size 1.5 1.5) (thickness 0.3)) (justify mirror))
   )
