File: EDA/PAL16R LART/PAL16R LART.kicad_pcb (KiCad board)
At the start: 2 copper layers, 40.6 x 47 mm, 6 parts, among them J1 Probe, U1 PINS, U2 DIP 20 ZIF

Commit message: minor fixes for production
Other:
- board text added: "JLCJLCJLCJLC"
Changed lines of the file:
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@@
   (general
     (thickness 1.6)
-    (drawings 17)
+    (drawings 18)
     (tracks 156)
     (zones 0)
@@
     (visible_elements FFFFFF7F)
     (pcbplotparams
-      (layerselection 0x010fc_ffffffff)
+      (layerselection 0x010e0_ffffffff)
       (usegerberextensions false)
       (usegerberattributes true)
@@
       (outputformat 1)
       (mirror false)
-      (drillshape 1)
+      (drillshape 0)
       (scaleselection 1)
       (outputdirectory ""))
@@
       (effects (font (size 1 1) (thickness 0.15)))
     )
-    (fp_text user %R (at 1.27 11.43 90) (layer F.Fab)
-      (effects (font (size 1 1) (thickness 0.15)))
-    )
     (fp_line (start 0 -1.27) (end 3.81 -1.27) (layer F.Fab) (width 0.1))
     (fp_line (start 3.81 -1.27) (end 3.81 24.13) (layer F.Fab) (width 0.1))
@@
     (fp_line (start 4.35 24.65) (end 4.35 -1.8) (layer F.CrtYd) (width 0.05))
     (fp_line (start 4.35 -1.8) (end -1.8 -1.8) (layer F.CrtYd) (width 0.05))
+    (fp_text user %R (at 1.27 11.43 90) (layer F.Fab)
+      (effects (font (size 1 1) (thickness 0.15)))
+    )
     (pad 20 thru_hole oval (at 2.54 22.86) (size 1.7 1.7) (drill 1) (layers *.Cu *.Mask)
       (net 12 /~OE))
@@
     )
   )
+  (gr_text JLCJLCJLCJLC (at 207 92.5 90) (layer F.SilkS)
+    (effects (font (size 1.5 1.5) (thickness 0.3)))
+  )
   (gr_text "C\n\nI2\n\nI3\n\nI4\n\nI5\n\nI6\n\nI7\n\nI8\n\nI9\n\nG" (at 177.165 92.71) (layer F.SilkS)

Commit message: PAL16R LART: v1.0.0
Connections:
- net /~OE renamed /~{OE}
Other:
- net class Default removed
- net class GND removed
- net class VCC removed
