File: EDA/Design68/ISO/341-0001_Matrix.kicad_sch (KiCad schematic)
At the start: 69 parts, among them SW1 1u, SW10 1u, SW11 1u, SW12 1u, SW13 1u, SW14 2u, SW15 1u, SW16 1.5u, SW17 1u, SW18 1u, SW19 1u, SW2 1u, SW20 1u, SW21 1u, SW22 1u, SW23 1u, SW24 1u, SW25 1u, SW26 1u, SW27 1u, SW28 1u, SW29 L shit, SW3 1u, SW30 1u, SW31 1.75u, SW32 1u, SW33 1u, SW34 1u, SW35 1u, SW36 1u, SW37 1u, SW38 1u, SW39 1u, SW4 1u, SW40 1u, SW41 1u, SW42 1u, SW43 1u, SW44 1u, SW45 1.25u, SW46 1u, SW47 1u, SW48 1u, SW49 1u, SW5 1u, SW50 1u, SW51 1u, SW52 1u, SW53 1u, SW54 1u, SW55 1u, SW56 1u, SW57 1.75u, SW58 1u, SW59 1u, SW6 1u, SW60 1.25u, SW61 1.25u, SW62 1.25u, SW63 6.25u, SW64 1u, SW65 1u, SW66 1u, SW67 1u, SW68 1u, SW69 1u, SW7 1u, SW8 1u, SW9 1u

Commit message: Preparing for ANSI, cleaning
Other:
- company: (none) -> lostwave
- title: (none) -> Design68 341-0001 ISO
Changed lines of the file:
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@@
 (kicad_sch (version 20230121) (generator eeschema)
   (paper "A4")
+  (title_block
+    (title "Design68 341-0001 ISO")
+    (date "2023-09-14")
+    (rev "1.0")
+    (company "lostwave")
+    (comment 1 "https://github.com/demik/oldworld/blob/master/EDA/Design68/README.md")
+  )
   (bus (pts (xy 25.4 190.5) (xy 38.1 190.5))
     (stroke (width 0) (type default))
