File: EDA/Design68/ISO/Design68.kicad_sch (KiCad schematic)
At the start: 19 parts, among them J3 Mini-DIN-4, J4 Wires, K1 KS88C0504 DIP Socket, Y1 4 MHz

Commit message: Preparing for ANSI, cleaning
Other:
- company: (none) -> lostwave
- title: (none) -> Design68 341-0001 ISO
Changed lines of the file:
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@@
   (paper "A4")
   (title_block
-    (date "2023-07-30")
+    (title "Design68 341-0001 ISO")
+    (date "2023-09-14")
+    (rev "1.0")
+    (company "lostwave")
+    (comment 1 "https://github.com/demik/oldworld/blob/master/EDA/Design68/README.md")
   )
   (junction (at 60.96 60.96) (diameter 0) (color 0 0 0 0)
