File: EDA/Design68/ISO/Mounting_Holes.kicad_sch (KiCad schematic)
At the start: 12 parts

Commit message: Preparing for ANSI, cleaning
Other:
- company: (none) -> lostwave
- title: (none) -> Design68 341-0001 ISO
Changed lines of the file:
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@@
 (kicad_sch (version 20230121) (generator eeschema)
   (paper "A4")
+  (title_block
+    (title "Design68 341-0001 ISO")
+    (date "2023-09-14")
+    (rev "1.0")
+    (company "lostwave")
+    (comment 1 "https://github.com/demik/oldworld/blob/master/EDA/Design68/README.md")
+  )
   (rectangle (start 38.1 38.1) (end 270.51 101.6)
     (stroke (width 0) (type default))
