File: EDA/ADBDB/ADBDB.kicad_pcb (KiCad board)
At the start: 2 copper layers, 100 x 50 mm, 40 parts, among them J1 Amphenol 61729, J2 Conn_01x04, J3 Mini-DIN-4, J4 Conn_01x03, J5 Mini-DIN-4, J6 Conn_01x04, J7 Conn_01x04, SW1 SW_DIP_x03, SW2 SW_DIP_x03, U1 PIC12F1840-IP, U2 PIC12F1840-IP, U3 PIC12F1840-IP, U5 NE555P

Commit message: ADBDB final touches
Parts:
- C1: value C -> 100nF
Other:
- board text added: "G ADB G Tx"
- board text added: "G CTS Rx Tx"
- board text removed: "G D Rx Tx"
- board text removed: "G adb G Tx"
Changed lines of the file:
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@@
   (title_block
     (title "ADBDB")
-    (date "2024-02-14")
+    (date "2024-02-16")
     (rev "1.1")
     (company "68kmla")
@@
         (effects (font (size 1 1) (thickness 0.15)))
     )
-    (fp_text value "C" (at 2.5 2.2) (layer "F.Fab")
+    (fp_text value "100nF" (at 2.5 2.2) (layer "F.Fab")
         (effects (font (size 1 1) (thickness 0.15)))
     )
@@
     (effects (font (size 1.5 1.5) (thickness 0.3) bold))
   )
-  (gr_text "G adb G  Tx" (at 115.316 75) (layer "F.SilkS")
+  (gr_text "G ADB G  Tx" (at 115.062 75) (layer "F.SilkS")
     (effects (font (size 1 1) (thickness 0.15)) (justify left bottom))
   )
@@
     (effects (font (size 1 1) (thickness 0.15)))
   )
-  (gr_text "G  D  Rx Tx" (at 152.5 75) (layer "F.SilkS")
+  (gr_text "G CTS Rx Tx" (at 152.5 75) (layer "F.SilkS")
     (effects (font (size 1 1) (thickness 0.15)) (justify left bottom))
   )
