File: EDA/ADBDB/Device.kicad_sch (KiCad schematic)
At the start: 8 parts, among them J2 Conn_01x04, J3 Mini-DIN-4, J4 Conn_01x03, U3 PIC12F1840-IP

Commit message: ADBDB final touches
Parts:
- C1: value C -> 100nF
Changed lines of the file:
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@@
   (title_block
     (title "ADBDB")
-    (date "2024-02-11")
+    (date "2024-02-16")
     (rev "1.1")
     (company "68kmla")
@@
       (effects (font (size 1.27 1.27)) (justify right))
     )
-    (property "Value" "C" (at 72.771 109.1621 0)
+    (property "Value" "100nF" (at 72.771 109.1621 0)
       (effects (font (size 1.27 1.27)) (justify right))
     )
