File: EDA/SIMM72BL/SIMM72BL.kicad_pcb (KiCad board)
At the start: 4 copper layers, 108 x 35.8 mm, 135 parts, among them J1 5822021-4, U1 SIMM-72, U10 74HC14, U2 74HC14, U3 74HC14, U4 74HC14, U5 74HC14, U6 74HC14, U7 74HC14, U8 74HC14, U9 74HC14

Commit message: SIMM72BL v1.2: fixed decoupling caps footprint & silkscreen
Parts:
- moved REF** 5.63 mm to (61.0, 107.0)
Other:
- board text removed: "JLCJLCJLCJLC"
